File: mk19-rp2040.kicad_pcb (KiCad board)
At the start: 2 copper layers, 41.8 x 77.6 mm, 43 parts, among them J1 USB_C_Receptacle_USB2.0, J5 Conn_01x02, U1 RP2040, U2 USBLC6-2P6, U3 XC6210B332MR-G, U4 USBLC6-2P6, U5 W25Q128JVS, Y1 Crystal_GND24

Commit message: starting on first pass at placing components
Parts:
- removed C2: 1µ, Capacitor_SMD:C_0603_1608Metric
- removed G*** (x4): LOGO, LOGO
- removed kibuzzard-61F01B61: G***, kibuzzard-61F01B61
- removed kibuzzard-6208EFFE: G***, kibuzzard-6208EFFE
- added 5WAY1: Conn_01x08_Socket, Connector_JST:JST_EH_S8B-EH_1x08_P2.50mm_Horizontal, F.Cu at (79.6, -91.9)
- added AUDIO1: Conn_01x03_Socket, Connector_JST:JST_EH_B3B-EH-A_1x03_P2.50mm_Vertical, F.Cu at (125.1, -42.7)
- added C15: CL31B105KBHNNNE, ct-kicad:C1206, F.Cu at (124.7, -78.6)
- added C16: CL31B105KBHNNNE, ct-kicad:C1206, F.Cu at (124.7, -74.9)
- added C17: 1µ, Capacitor_SMD:C_0402_1005Metric, F.Cu at (139.2, -55.3)
- added C18: 100nF, ct-kicad:C0402, F.Cu at (137.7, -32.4)
- added C19: 100nF, ct-kicad:C0402, F.Cu at (137.7, -29.9)
- added C20: CL31B105KBHNNNE, ct-kicad:C1206, F.Cu at (124.7, -71.3)
- added C21: CL31B105KBHNNNE, ct-kicad:C1206, F.Cu at (124.7, -67.6)
- added C22: CL31B105KBHNNNE, ct-kicad:C1206, F.Cu at (124.7, -64.0)
- added C23: 100nF, ct-kicad:C0402, F.Cu at (137.7, -27.5)
- added C24: 100nF, ct-kicad:C0402, F.Cu at (137.7, -25.0)
- added C25: 100nF, ct-kicad:C0402, F.Cu at (137.7, -22.5)
- added C26: 100nF, ct-kicad:C0402, F.Cu at (137.7, -20.0)
- added C27: 10u, Capacitor_SMD:C_0805_2012Metric, F.Cu at (123.8, -18.1)
- added COL1: Conn_01x08_Socket, Connector_JST:JST_EH_S8B-EH_1x08_P2.50mm_Horizontal, F.Cu at (79.6, -81.5)
- added COL2: Conn_01x08_Socket, Connector_JST:JST_EH_S8B-EH_1x08_P2.50mm_Horizontal, F.Cu at (79.6, -71.1)
- added COL_CS_MOS1: 2N7002, ct-kicad:SOT-23-3_L2.9-W1.3-P1.90-LS2.4-BR, F.Cu at (128.4, -21.7)
- added CYBOARD-MACRO1: HC-FPC-05-10-16RLTAG, ct-kicad:FPC-SMD_16P-P0.50_HCTL_HC-FPC-05-10-16RLTAG, F.Cu at (115.7, -60.4)
- added CYBOARD-MAIN1: ECT818001569, ct-kicad:FPC-SMD_ECT818001569, F.Cu at (115.3, -55.8)
- added D3: B5817, Diode_SMD:D_SOD-323, F.Cu at (135.6, -54.8)
- added D4: SMF5_0CA_C364279, ct-kicad:SOD-123FL_L2.8-W1.8-LS3.7-BI, F.Cu at (134.8, -51.2)
- added F2: Polyfuse, Fuse:Fuse_0603_1608Metric, F.Cu at (123.6, -60.7)
- added F3: MF-NSMF075-2, ct-kicad:F1206, F.Cu at (136.3, -58.2)
- added FAL1: Conn_01x08_Socket, Connector_JST:JST_EH_S8B-EH_1x08_P2.50mm_Horizontal, F.Cu at (79.6, -60.8)
- added FAL2: Conn_01x08_Socket, Connector_JST:JST_EH_S8B-EH_1x08_P2.50mm_Horizontal, F.Cu at (79.6, -50.4)
- added FB2: FerriteBead_Small, Inductor_SMD:L_0603_1608Metric, F.Cu at (123.6, -58.2)
- added FB3: FerriteBead_Small, Inductor_SMD:L_0603_1608Metric, F.Cu at (123.6, -55.7)
- added H1: MountingHole, MountingHole:MountingHole_3.2mm_M3_Pad_Via, F.Cu at (132.9, 53.1)
- added H2: MountingHole, MountingHole:MountingHole_3.2mm_M3_Pad_Via, F.Cu at (252.9, 53.1)
- added H3: MountingHole, MountingHole:MountingHole_3.2mm_M3_Pad_Via, F.Cu at (132.9, 128.1)
- added H4: MountingHole, MountingHole:MountingHole_3.2mm_M3_Pad_Via, F.Cu at (252.9, 128.1)
- added J10: Conn_01x02, drawings:PinHeader_1x02_P1.27mm_Vertical, F.Cu at (106.3, -19.8)
- added J11: Conn_01x03_Socket, Connector_PinHeader_2.54mm:PinHeader_1x03_P2.54mm_Vertical, F.Cu at (138.2, -97.3)
- added J12: USB_C_Receptacle_USB2.0, drawings:GT-USB-7014C, F.Cu at (128.7, -90.7)
- added J13: USB_C_Receptacle_USB2.0, drawings:GT-USB-7014C, F.Cu at (128.7, -81.0)
- added J2: Conn_01x02_Socket, Connector_JST:JST_EH_B2B-EH-A_1x02_P2.50mm_Vertical, F.Cu at (104.2, -97.0)
- added J3: Conn_01x02_Socket, Connector_JST:JST_EH_B2B-EH-A_1x02_P2.50mm_Vertical, F.Cu at (104.2, -91.2)
- added J4: Conn_01x02_Socket, Connector_JST:JST_EH_B2B-EH-A_1x02_P2.50mm_Vertical, F.Cu at (104.2, -85.3)
- added J6: Conn_01x02_Socket, Connector_JST:JST_EH_B2B-EH-A_1x02_P2.50mm_Vertical, F.Cu at (104.2, -79.5)
- added J7: Conn_01x02_Socket, Connector_JST:JST_EH_B2B-EH-A_1x02_P2.50mm_Vertical, F.Cu at (104.2, -73.6)
- added J8: Conn_01x02_Socket, Connector_JST:JST_EH_B2B-EH-A_1x02_P2.50mm_Vertical, F.Cu at (104.2, -67.8)
- added J9: Conn_01x02_Socket, Connector_JST:JST_EH_B2B-EH-A_1x02_P2.50mm_Vertical, F.Cu at (104.2, -61.9)
- added L1: MPZ2012S101AT000, ct-kicad:L0805, F.Cu at (134.6, -47.8)
- added LED-LVL1: SN74LVC1T45DRL, ct-kicad:SOT-563_L1.6-W1.2-P0.50-LS1.6-BR, F.Cu at (138.7, -47.8)
- added LOGO1: **REF, ct-kicad:awesome-logo, F.Cu at (252.4, -10.9)
- added LOGO2: **REF, ct-kicad:qmk-lite, F.Cu at (209.1, -19.8)
- added LOGO3: **REF, ct-kicad:mk19-qr-logo-12mm, F.Cu at (261.0, -13.9)
- added LOGO4: **REF, ct-kicad:awesome-logo, F.Cu at (245.0, -11.0)
- added LOGO5: **REF, ct-kicad:qmk-lite, F.Cu at (235.8, -20.1)
- added LOGO6: **REF, ct-kicad:cyboard-logo-10mm, F.Cu at (237.3, -11.9)
- added LOGO7: **REF, ct-kicad:cyboard-logo-10mm, F.Cu at (229.1, -12.7)
- added MOSFET1: AO3401A_C347476, ct-kicad:SOT-23_L2.9-W1.3-P1.90-LS2.4-BR, F.Cu at (123.7, -21.8)
- added PWM1: Conn_01x08_Socket, Connector_JST:JST_EH_S8B-EH_1x08_P2.50mm_Horizontal, F.Cu at (79.6, -40.0)
- added PWR-EXT-IN1: Conn_01x02_Socket, Connector_JST:JST_EH_B2B-EH-A_1x02_P2.50mm_Vertical, F.Cu at (104.2, -56.1)
- added PWR-OUT1: Conn_01x03_Socket, Connector_JST:JST_EH_B3B-EH-A_1x03_P2.50mm_Vertical, F.Cu at (125.1, -36.8)
- added PWR-OUT2: Conn_01x03_Socket, Connector_PinSocket_2.54mm:PinSocket_1x03_P2.54mm_Vertical, F.Cu at (123.9, -31.3)
- added PWR-OUT3: Conn_01x03_Socket, Connector_PinSocket_2.54mm:PinSocket_1x03_P2.54mm_Vertical, F.Cu at (128.5, -31.3)
- added R13: 4.7k, ct-kicad:R1206, F.Cu at (136.5, -43.6)
- added R14: 4.7k, ct-kicad:R1206, F.Cu at (136.5, -40.2)
- added R15: 1206W4F1002T5E, ct-kicad:R1206, F.Cu at (136.5, -36.7)
- added R16: 4D03WGJ0103T5E, ct-kicad:RES-ARRAY-SMD_0603-8P-L3.2-W1.6-BL, F.Cu at (133.5, -31.5)
- added R17: 4D03WGJ0103T5E, ct-kicad:RES-ARRAY-SMD_0603-8P-L3.2-W1.6-BL, F.Cu at (133.5, -27.4)
- added R18: 4D03WGJ0103T5E, ct-kicad:RES-ARRAY-SMD_0603-8P-L3.2-W1.6-BL, F.Cu at (133.5, -23.3)
- added R19: 4D03WGJ0103T5E, ct-kicad:RES-ARRAY-SMD_0603-8P-L3.2-W1.6-BL, F.Cu at (133.5, -19.2)
- added REG-COL1: MC74HC589ADR2G, ct-kicad:SOIC-16_L9.9-W3.9-P1.27-LS6.0-BL, F.Cu at (116.0, -95.4)
- added REG-COL2: MC74HC589ADR2G, ct-kicad:SOIC-16_L9.9-W3.9-P1.27-LS6.0-BL, F.Cu at (116.0, -86.4)
- added REG-ROW1: 74HC595D, ct-kicad:SOIC-16_L9.9-W3.9-P1.27-LS6.0-BL, F.Cu at (116.0, -77.3)
- added REG-ROW2: 74HC595D, ct-kicad:SOIC-16_L9.9-W3.9-P1.27-LS6.0-BL, F.Cu at (116.0, -68.3)
- added ROW1: Conn_01x08_Socket, Connector_JST:JST_EH_S8B-EH_1x08_P2.50mm_Horizontal, F.Cu at (79.6, -29.6)
- added ROW2: Conn_01x08_Socket, Connector_JST:JST_EH_S8B-EH_1x08_P2.50mm_Horizontal, F.Cu at (79.6, -19.2)
- added T1: Conn_01x01_Socket, Connector_Pin:Pin_D1.0mm_L10.0mm, F.Cu at (137.9, -87.9)
- added T2: Conn_01x01_Socket, Connector_Pin:Pin_D1.0mm_L10.0mm, F.Cu at (137.9, -83.9)
- added U10: 1N4148W_C81598, ct-kicad:SOD-123F_L2.7-W1.6-LS3.8-RD, F.Cu at (130.6, -66.6)
- added U11: 1N4148W_C81598, ct-kicad:SOD-123F_L2.7-W1.6-LS3.8-RD, F.Cu at (130.6, -62.8)
- added U12: 1N4148W_C81598, ct-kicad:SOD-123F_L2.7-W1.6-LS3.8-RD, F.Cu at (130.6, -59.1)
- added U13: 1N4148W_C81598, ct-kicad:SOD-123F_L2.7-W1.6-LS3.8-RD, F.Cu at (130.6, -55.3)
- added U6: 8_01A0_008200, ct-kicad:FPC-SMD_8P-P0.50_8.01A0.008200, F.Cu at (113.6, -29.1)
- added U7: 8_01A0_008200, ct-kicad:FPC-SMD_8P-P0.50_8.01A0.008200, F.Cu at (113.6, -21.7)
- added U8: USBLC6-2P6, Package_TO_SOT_SMD:SOT-666, F.Cu at (102.7, -19.2)
- added U9: 1N4148W_C81598, ct-kicad:SOD-123F_L2.7-W1.6-LS3.8-RD, F.Cu at (130.6, -70.3)
- C1: value 1µ -> 10u; footprint Capacitor_SMD:C_0603_1608Metric -> Capacitor_SMD:C_0805_2012Metric
- moved U2 114.0 mm to (103.6, -24.5), turned to 0 degrees
- moved J1 105.5 mm to (192.2, 48.1), turned to 180 degrees
- moved FB1 95.1 mm to (195.9, 72.2)
- moved R4 95.0 mm to (199.4, 71.9), turned to 0 degrees
- moved R5 89.9 mm to (199.4, 73.9), turned to 0 degrees
- moved U4 88.5 mm to (191.9, 72.8)
- moved D2 45.2 mm to (196.2, 99.8)
- moved C1 45.2 mm to (199.0, 103.4)
- moved C10 45.2 mm to (185.5, 104.7)
- moved C11 45.2 mm to (202.2, 108.3)
- moved C12 45.2 mm to (192.7, 108.4)
- moved C13 45.2 mm to (202.9, 112.7)
- moved C14 45.2 mm to (199.6, 117.9)
- moved C3 45.2 mm to (195.2, 120.9)
- moved C4 45.2 mm to (197.2, 120.9)
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Connections:
- D1 pad 2: /LED -> +5V
- FB1 pad 1: /Gnd_daughter -> GND
- J1 pad A1: /Gnd_daughter -> GND
- J1 pad A12: /Gnd_daughter -> GND
- J1 pad A4: /Vbus_daughter -> /Serial_VBUS
- J1 pad A6: /D+_daughter -> USB-MAIN_+
- J1 pad A7: /D-_daughter -> USB-MAIN_-
- J1 pad A9: /Vbus_daughter -> /Serial_VBUS
- J1 pad B1: /Gnd_daughter -> GND
- J1 pad B12: /Gnd_daughter -> GND
- J1 pad B4: /Vbus_daughter -> /Serial_VBUS
- J1 pad B6: /D+_daughter -> USB-MAIN_+
- J1 pad B7: /D-_daughter -> USB-MAIN_-
- J1 pad B9: /Vbus_daughter -> /Serial_VBUS
- J5 pad 1: GND -> Net-(J5-Pin_1)
- J5 pad 2: Net-(J5-Pin_2) -> GND
- R2 pad 1: /~{RESET} -> +3V3
- R2 pad 2: +3V3 -> Net-(J10-Pin_1)
- R3 pad 1: Net-(J5-Pin_2) -> Net-(J5-Pin_1)
- R4 pad 2: /Gnd_daughter -> GND
- R5 pad 2: /Gnd_daughter -> GND
- R6 pad 1: /D+ -> USB-MAIN_+
- R7 pad 1: /D- -> USB-MAIN_-
- U1 pad 11: col6_l -> fal2-r2
- U1 pad 12: row5_l -> Net-(LED-LVL1-A)
- U1 pad 13: unconnected-(U1-GPIO10-Pad13) -> SPI1_CLK
- U1 pad 14: unconnected-(U1-GPIO11-Pad14) -> SPI1_MOSI
- U1 pad 15: unconnected-(U1-GPIO12-Pad15) -> SPI1_MISO
- U1 pad 16: unconnected-(U1-GPIO13-Pad16) -> COL_CS
- U1 pad 17: unconnected-(U1-GPIO14-Pad17) -> COL_LATCH
- U1 pad 18: split_hand_l -> ROW_CS
- U1 pad 2: rgb_r -> Serial-RX
- U1 pad 24: unconnected-(U1-SWCLK-Pad24) -> Net-(J11-Pin_3)
- U1 pad 25: unconnected-(U1-SWD-Pad25) -> Net-(J11-Pin_2)
- U1 pad 26: /~{RESET} -> Net-(J10-Pin_1)
- U1 pad 27: ss_l -> PMW_CS
- U1 pad 28: /LED -> LCD1_CS
- U1 pad 29: unconnected-(U1-GPIO18-Pad29) -> LCD2_CS
- U1 pad 3: serial_l -> Serial-RX
- U1 pad 30: /VBUS_DET -> LCD_BL
- U1 pad 31: miso_l -> LCD_DC
- U1 pad 32: col3_l -> LCD_RST
- U1 pad 34: sc_l -> unconnected-(U1-GPIO22-Pad34)
- U1 pad 35: mosi_l -> unconnected-(U1-GPIO23-Pad35)
- U1 pad 38: row2_l -> unconnected-(U1-GPIO26_ADC0-Pad38)
- U1 pad 39: col1_l -> unconnected-(U1-GPIO27_ADC1-Pad39)
- U1 pad 4: unconnected-(U1-GPIO2-Pad4) -> split_hand
- U1 pad 40: col2_l -> unconnected-(U1-GPIO28_ADC2-Pad40)
- U1 pad 41: row1_l -> /VBUS_DET
- U1 pad 5: unconnected-(U1-GPIO3-Pad5) -> rkjxt-a
- U1 pad 6: row4_l -> rkjxt-b
- U1 pad 7: row3_l -> fal1-r1
- U1 pad 8: col4_l -> fal1-r2
- U1 pad 9: col5_l -> fal2-r1
- U2 pad 1: serial_l -> LED_SCREEN_DO
- U2 pad 3: unconnected-(U2-I/O2-Pad3) -> LED_SCREEN_DI
- U2 pad 4: unconnected-(U2-I/O2-Pad4) -> LED_SCREEN_DI
- U2 pad 5: +3V3 -> +5V
- U2 pad 6: serial_l -> LED_SCREEN_DO
- U4 pad 1: /D-_daughter -> USB-MAIN_-
- U4 pad 2: /Gnd_daughter -> GND
- U4 pad 3: /D+_daughter -> USB-MAIN_+
- U4 pad 4: /D+_daughter -> USB-MAIN_+
- U4 pad 5: /Vbus_daughter -> +5V
- U4 pad 6: /D-_daughter -> USB-MAIN_-
Routing:
- net mosi_l: track 46.1 -> 0.00 mm
- net sc_l: track 43.3 -> 0.00 mm
- net miso_l: track 42.2 -> 0.00 mm, vias 1 -> 0
- net /~{RESET}: track 39.9 -> 0.00 mm, vias 1 -> 0
- net +3V3: track 122.9 -> 85.7 mm, vias 3 -> 4
- net ss_l: track 36.5 -> 0.00 mm, vias 1 -> 0
- net row2_l: track 35.1 -> 0.00 mm, vias 1 -> 0
- net serial_l: track 33.6 -> 0.00 mm, vias 2 -> 0
- net col1_l: track 33.0 -> 0.00 mm, vias 1 -> 0
- net col2_l: track 31.0 -> 0.00 mm, vias 1 -> 0
- net Serial-RX: track 0.00 -> 30.0 mm, vias 0 -> 2
- net /D-_daughter: track 29.2 -> 0.00 mm, vias 2 -> 0
- net row1_l: track 28.7 -> 0.00 mm, vias 1 -> 0
- net /Vbus_daughter: track 27.1 -> 0.00 mm, vias 3 -> 0
- net col3_l: track 25.6 -> 0.00 mm, vias 1 -> 0
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- removed copper zone on B.Cu, net /Gnd_daughter
- removed copper zone on F.Cu, net /Gnd_daughter
Other:
- board size 41.8 x 77.6 mm -> 130 x 85 mm
- board text removed: "3.3V"
- board text removed: "C1"
- board text removed: "C2"
- board text removed: "C3"
- board text removed: "C4"
- board text removed: "C5"
- board text removed: "C6"
- board text removed: "CERN OHL-S v2"
- board text removed: "Compatible with splinky v3"
- board text removed: "DESIGN BY QUENTIN LEBASTARD BASTARDKB 2023"
- board text removed: "GND"
- board text removed: "MATRIX"
- board text removed: "MI"
- board text removed: "MO"
- board text removed: "R1"
- board text removed: "R2"
- board text removed: "R3"
- board text removed: "R4"
- board text removed: "R5"
- board text removed: "REV1.4"
- board text removed: "RGB"
- board text removed: "SC"
- board text removed: "SS"
- board text removed: "TRCK"
- board text removed: "USB board on THIS side for Left"
- board text removed: "USB board on THIS side for Right"
- board text removed: "V-CUT"
- board text removed: "mk19-rp2040 REV 1.4"
- board text removed: "this side not visible"

Commit message: some bad footprints, other fixes
Parts:
- removed J2, J4, J6: Conn_01x02_Socket, Connector_JST:JST_EH_B2B-EH-A_1x02_P2.50mm_Vertical
- added JP1: SolderJumper_3_Open, Jumper:SolderJumper-3_P1.3mm_Open_Pad1.0x1.5mm, F.Cu at (68.9, -82.3)
- added JP2: SolderJumper_3_Open, Jumper:SolderJumper-3_P1.3mm_Open_Pad1.0x1.5mm, F.Cu at (68.9, -78.4)
- added JP3: SolderJumper_3_Open, Jumper:SolderJumper-3_P1.3mm_Open_Pad1.0x1.5mm, F.Cu at (68.9, -74.6)
- added R12: 10k, Resistor_SMD:R_0402_1005Metric, F.Cu at (51.3, -70.9)
- added R20: 10k, Resistor_SMD:R_0402_1005Metric, F.Cu at (51.3, -68.9)
- added T10: Conn_01x01_Socket, Connector_Pin:Pin_D1.0mm_L10.0mm, F.Cu at (60.0, -82.0)
- added T11: Conn_01x01_Socket, Connector_Pin:Pin_D1.0mm_L10.0mm, F.Cu at (60.0, -78.0)
- added T12: Conn_01x01_Socket, Connector_Pin:Pin_D1.0mm_L10.0mm, F.Cu at (60.0, -73.9)
- added T13: Conn_01x01_Socket, Connector_Pin:Pin_D1.0mm_L10.0mm, F.Cu at (64.0, -82.0)
- added T14: Conn_01x01_Socket, Connector_Pin:Pin_D1.0mm_L10.0mm, F.Cu at (64.0, -78.0)
- added T15: Conn_01x01_Socket, Connector_Pin:Pin_D1.0mm_L10.0mm, F.Cu at (64.0, -73.9)
- added T3: Conn_01x01_Socket, Connector_Pin:Pin_D1.0mm_L10.0mm, F.Cu at (51.9, -82.0)
- added T5: Conn_01x01_Socket, Connector_Pin:Pin_D1.0mm_L10.0mm, F.Cu at (51.9, -78.0)
- added T6: Conn_01x01_Socket, Connector_Pin:Pin_D1.0mm_L10.0mm, F.Cu at (51.9, -73.9)
- added T7: Conn_01x01_Socket, Connector_Pin:Pin_D1.0mm_L10.0mm, F.Cu at (55.9, -82.0)
- added T8: Conn_01x01_Socket, Connector_Pin:Pin_D1.0mm_L10.0mm, F.Cu at (55.9, -78.0)
- added T9: Conn_01x01_Socket, Connector_Pin:Pin_D1.0mm_L10.0mm, F.Cu at (55.9, -73.9)
- added U14: 1N4148W_C81598, ct-kicad:SOD-123F_L2.7-W1.6-LS3.8-RD, F.Cu at (68.8, -71.0)
- added U15: 1N4148W_C81598, ct-kicad:SOD-123F_L2.7-W1.6-LS3.8-RD, F.Cu at (68.8, -67.3)
- added VANILED1: Conn_01x08_Socket, Connector_JST:JST_XH_B8B-XH-AM_1x08_P2.50mm_Vertical, F.Cu at (53.3, -88.5)
- 5WAY1, COL1, COL2, FAL1, FAL2, PWM1, ROW1, ROW2: footprint Connector_JST:JST_EH_S8B-EH_1x08_P2.50mm_Horizontal -> Connector_JST:JST_XH_S8B-XH-A_1x08_P2.50mm_Horizontal
- AUDIO1, PWR-OUT1: footprint Connector_JST:JST_EH_B3B-EH-A_1x03_P2.50mm_Vertical -> Connector_JST:JST_XH_B3B-XH-AM_1x03_P2.50mm_Vertical
- J1, J12, J13: footprint drawings:GT-USB-7014C -> ct-kicad:USB-C-SMD_12P-P0.50-H-F_TYPE-C-31-M-14
- J11: footprint Connector_PinHeader_2.54mm:PinHeader_1x03_P2.54mm_Vertical -> Connector_JST:JST_XH_B3B-XH-AM_1x03_P2.50mm_Vertical
- J3, J7, J8, J9, PWR-EXT-IN1: footprint Connector_JST:JST_EH_B2B-EH-A_1x02_P2.50mm_Vertical -> Connector_JST:JST_XH_B2B-XH-AM_1x02_P2.50mm_Vertical
- PWR-OUT3: footprint Connector_PinSocket_2.54mm:PinSocket_1x03_P2.54mm_Vertical -> Connector_JST:JST_XH_B3B-XH-AM_1x03_P2.50mm_Vertical
- moved J13 169.9 mm to (232.9, 53.2), turned to 180 degrees
- moved J12 166.7 mm to (212.9, 53.2), turned to 180 degrees
- moved F1 38.1 mm to (189.7, 58.7)
- moved U1 37.4 mm to (193.0, 74.6)
- moved U3 37.4 mm to (194.6, 63.4)
- moved C1 37.4 mm to (194.6, 66.3)
- moved C10 37.4 mm to (181.1, 67.6)
- moved C11 37.4 mm to (197.7, 71.2)
- moved C12 37.4 mm to (188.3, 71.3)
- moved C13 37.4 mm to (198.4, 75.6)
- moved C14 37.4 mm to (195.1, 80.8)
- moved C3 37.4 mm to (190.7, 83.8)
- moved C4 37.4 mm to (192.7, 83.8)
- moved C5 37.4 mm to (198.7, 71.2)
- moved C6 37.4 mm to (196.7, 69.1)
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Connections:
- 5WAY1 pad 1: Net-(5WAY1-Pin_1) -> rkjxt-b
- 5WAY1 pad 2: Net-(5WAY1-Pin_2) -> rkjxt-a
- AUDIO1 pad 2: GPIO6 -> AUDIO
- CYBOARD-MACRO1 pad 1: VCC -> +5V
- CYBOARD-MACRO1 pad 10: row9 -> row3
- CYBOARD-MACRO1 pad 2: VCC -> +5V
- CYBOARD-MACRO1 pad 3: VCC -> +5V
- CYBOARD-MACRO1 pad 4: VCC -> +5V
- CYBOARD-MACRO1 pad 5: col8 -> col6
- CYBOARD-MACRO1 pad 6: col9 -> col7
- CYBOARD-MACRO1 pad 7: col10 -> col8
- CYBOARD-MACRO1 pad 8: col11 -> col9
- CYBOARD-MACRO1 pad 9: row8 -> row2
- CYBOARD-MAIN1 pad 13: VCC -> +5V
- CYBOARD-MAIN1 pad 14: VCC -> +5V
- CYBOARD-MAIN1 pad 15: VCC -> +5V
- CYBOARD-MAIN1 pad 16: VCC -> +5V
- F2 pad 1: Net-(PWR-OUT3-Pin_2) -> Net-(JP1-A)
- FAL1 pad 2: VCC -> +5V
- FAL1 pad 6: col6 -> Net-(FAL1-Pin_6)
- FAL2 pad 2: VCC -> +5V
- FAL2 pad 4: LED_SLATS_BIG_DI -> LED_KEYBAR_DI
- FAL2 pad 6: col7 -> Net-(FAL2-Pin_6)
- J3 pad 2: LED_SLATS_SM_DI -> LED_SCREEN_DI
- MOSFET1 pad 2: VCC -> Net-(JP2-B)
- PWR-OUT1 pad 3: VCC -> +5V
- PWR-OUT2 pad 3: VCC -> +5V
- PWR-OUT3 pad 2: Net-(PWR-OUT3-Pin_2) -> Net-(JP1-C)
- PWR-OUT3 pad 3: VCC -> +5V
- R13 pad 1: Net-(5WAY1-Pin_2) -> rkjxt-a
- R13 pad 2: rkjxt-a -> +5V
- R14 pad 1: Net-(5WAY1-Pin_1) -> rkjxt-b
- R14 pad 2: rkjxt-b -> +5V
- U1 pad 34: unconnected-(U1-GPIO22-Pad34) -> VANILED_SIG1
- U1 pad 35: unconnected-(U1-GPIO23-Pad35) -> VANILED_SIG2
- U1 pad 36: unconnected-(U1-GPIO24-Pad36) -> VANILED_SIG3
- U1 pad 37: unconnected-(U1-GPIO25-Pad37) -> VANILED_SIG3
- U1 pad 38: unconnected-(U1-GPIO26_ADC0-Pad38) -> AUDIO
- U1 pad 39: unconnected-(U1-GPIO27_ADC1-Pad39) -> Net-(T5-Pin_1)
- U1 pad 40: unconnected-(U1-GPIO28_ADC2-Pad40) -> Net-(T6-Pin_1)
Routing:
- net VANILED_SIG2: track 0.00 -> 7.15 mm
- net unconnected-(U1-GPIO23-Pad35): track 7.15 -> 0.00 mm
- net VANILED_SIG1: track 0.00 -> 6.89 mm
- net unconnected-(U1-GPIO22-Pad34): track 6.89 -> 0.00 mm
- net Net-(T6-Pin_1): track 0.00 -> 4.14 mm
- net unconnected-(U1-GPIO28_ADC2-Pad40): track 4.14 -> 0.00 mm
- net AUDIO: track 0.00 -> 3.65 mm
- net unconnected-(U1-GPIO26_ADC0-Pad38): track 3.65 -> 0.00 mm
- net unconnected-(U1-GPIO27_ADC1-Pad39): track 3.62 -> 0.00 mm
- net Net-(T5-Pin_1): track 0.00 -> 3.62 mm
- net Net-(D2-A): track 2.53 -> 3.47 mm
- net VBUS: track 16.7 -> 17.4 mm
- removed copper zone on F.Cu, net +3V3

Commit message: progress update
Parts:
- moved J13 90.0 mm to (142.9, 53.2)
- moved C10 4.37 mm to (181.7, 71.9)
- moved C13 4.37 mm to (199.0, 79.9)
- moved C6 4.37 mm to (197.3, 73.4)
- moved C9 4.37 mm to (188.5, 81.4)
- moved D2 4.37 mm to (192.4, 67.0)
- moved F1 4.37 mm to (190.3, 63.0)
- moved R10 4.37 mm to (197.3, 72.3)
- moved R2 4.37 mm to (198.6, 83.8)
- moved U1 4.37 mm to (193.6, 78.9)
- moved Y1 4.37 mm to (192.0, 85.8)
- moved C1 4.37 mm to (195.1, 70.6)
- moved C11 4.37 mm to (198.3, 75.5)
- moved C12 4.37 mm to (188.9, 75.6)
- moved C14 4.37 mm to (195.7, 85.1)
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Connections:
- FB1 pad 2: Net-(J1-SHIELD) -> Net-(FB1-Pad2)
- FB3 pad 2: Net-(J13-SHIELD) -> Net-(J13-DN1)
- J1 pad A1B12: (no net) -> GND
- J1 pad A4B9: (no net) -> VBUS
- J1 pad A6: USB-MAIN_+ -> USB-MAIN_-
- J1 pad A7: USB-MAIN_- -> USB-MAIN_+
- J1 pad B1A12: (no net) -> GND
- J1 pad B4A9: (no net) -> VBUS
- J1 pad B6: USB-MAIN_+ -> USB-MAIN_-
- J1 pad B7: USB-MAIN_- -> USB-MAIN_+
- J1 pad S: (no net) -> Net-(FB1-Pad2)
- J12 pad A1B12: (no net) -> GND
- J12 pad A4B9: (no net) -> /Serial_VBUS
- J12 pad A6: Split_Comms_TX -> Split_Comms_RX
- J12 pad A7: Split_Comms_RX -> Split_Comms_TX
- J12 pad B1A12: (no net) -> GND
- J12 pad B4A9: (no net) -> /Serial_VBUS
- J12 pad B6: Split_Comms_TX -> Split_Comms_RX
- J12 pad B7: Split_Comms_RX -> Split_Comms_TX
- J12 pad S: (no net) -> Net-(J12-SHIELD)
- J13 pad A1B12: (no net) -> GND
- J13 pad A4B9: (no net) -> /Serial_VBUS
- J13 pad A6: LED_SCREEN_DI -> LED_SCREEN_DO
- J13 pad A7: LED_SCREEN_DO -> LED_SCREEN_DI
- J13 pad B1A12: (no net) -> GND
- J13 pad B4A9: (no net) -> /Serial_VBUS
- J13 pad B6: LED_SCREEN_DI -> LED_SCREEN_DO
- J13 pad B7: LED_SCREEN_DO -> LED_SCREEN_DI
- J13 pad S: (no net) -> Net-(J13-DN1)
Routing:
- net +3V3: track 85.7 -> 87.3 mm
Other:
- outline, holes or cut-outs redrawn

Commit message: fixes
Parts:
- moved J13 30.0 mm to (172.9, 53.2)
Changed lines of the file:
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@@
 			)
 		)
+		(sheetname "Root")
+		(sheetfile "mk19-rp2040.kicad_sch")
 		(attr through_hole)
 		(fp_line
@@
 	(footprint "ct-kicad:USB-C-SMD_12P-P0.50-H-F_TYPE-C-31-M-14"
 		(layer "F.Cu")
-		(at 142.91 53.25 180)
+		(at 172.91 53.25 180)
 		(descr "USB-C-SMD_12P-P0.50-H-F_TYPE-C-31-M-14 footprint")
 		(tags "USB-C-SMD_12P-P0.50-H-F_TYPE-C-31-M-14 footprint C223907")
@@
 			)
 		)
+		(sheetname "Root")
+		(sheetfile "mk19-rp2040.kicad_sch")
 		(attr through_hole)
 		(fp_line
@@
 			)
 		)
+		(sheetname "Root")
+		(sheetfile "mk19-rp2040.kicad_sch")
 		(attr through_hole)
 		(fp_line

Commit message: getting close to having the rp2040 traced
Parts:
- removed 5WAY1: Conn_01x08_Socket, Connector_JST:JST_XH_S8B-XH-A_1x08_P2.50mm_Horizontal
- removed T8: Conn_01x01_Socket, Connector_Pin:Pin_D1.0mm_L10.0mm
- added J2: Conn_01x03_Socket, Connector_JST:JST_XH_S3B-XH-A_1x03_P2.50mm_Horizontal, F.Cu at (167.1, 31.9)
- added J4: Conn_01x06_Socket, Connector_JST:JST_XH_S6B-XH-A_1x06_P2.50mm_Horizontal, F.Cu at (167.1, 18.4)
- moved T5 220.3 mm to (209.2, 76.2)
- moved T6 215.3 mm to (209.3, 73.0)
- moved J5 205.0 mm to (49.7, -63.9), turned to 0 degrees
- moved D1 23.6 mm to (195.3, 63.8), turned to 180 degrees
- moved R1 22.5 mm to (197.2, 63.8)
- moved ROW2 20.5 mm to (78.7, 1.31)
- moved R3 14.6 mm to (177.0, 75.4), turned to -90 degrees
- moved R11 14.4 mm to (198.5, 58.5), turned to 0 degrees
- moved C1 13.5 mm to (185.4, 61.2), turned to 90 degrees
- moved R10 12.9 mm to (198.5, 59.5)
- moved T1 9.64 mm to (143.0, -79.8)
- moved T2 9.64 mm to (143.0, -75.7)
- moved U3 9.04 mm to (186.3, 65.8), turned to -90 degrees
- moved R5 7.65 mm to (191.2, 58.5), turned to -90 degrees
- moved D2 7.55 mm to (187.4, 61.3)
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Connections:
- J13 pad A4B9: /Serial_VBUS -> +5V
- J13 pad B4A9: /Serial_VBUS -> +5V
- U1 pad 2: Serial-RX -> Serial-TX
- U1 pad 37: VANILED_SIG3 -> VANILED_SIG4
- U1 pad 40: Net-(T6-Pin_1) -> /VBUS_DET
- U1 pad 41: /VBUS_DET -> Net-(T6-Pin_1)
Routing:
- net GND: track 24.4 -> 72.8 mm, vias 22 -> 32
- net +3V3: track 87.3 -> 109.2 mm, vias 4 -> 10
- net split_hand: track 0.00 -> 15.5 mm, vias 0 -> 1
- net Serial-RX: track 30.0 -> 14.6 mm, vias 2 -> 1
- net rkjxt-a: track 0.00 -> 15.2 mm
- net PMW_CS: track 4.44 -> 19.5 mm, vias 1 -> 2
- net USB-MAIN_+: track 5.37 -> 19.5 mm, vias 1 -> 2
- net Serial-TX: track 0.00 -> 13.5 mm, vias 0 -> 1
- net Net-(LED-LVL1-A): track 8.24 -> 19.7 mm, vias 0 -> 2
- net fal2-r2: track 8.47 -> 19.8 mm, vias 0 -> 2
- net Net-(T5-Pin_1): track 3.62 -> 14.9 mm, vias 0 -> 1
- net Net-(T6-Pin_1): track 4.14 -> 14.9 mm, vias 0 -> 1
- net COL_LATCH: track 0.00 -> 9.04 mm, vias 0 -> 1
- net Net-(J11-Pin_2): track 0.00 -> 8.99 mm, vias 0 -> 3
- net USB-MAIN_-: track 9.91 -> 18.6 mm, vias 1 -> 5
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Other:
- outline, holes or cut-outs redrawn

Commit message: more progress
Parts:
- AUDIO1, J11, PWR-OUT1: footprint Connector_JST:JST_XH_B3B-XH-AM_1x03_P2.50mm_Vertical -> Connector_JST:JST_XH_B3B-XH-A_1x03_P2.50mm_Vertical
- COL1, COL2, ROW1, ROW2: footprint Connector_JST:JST_XH_S8B-XH-A_1x08_P2.50mm_Horizontal -> Connector_JST:JST_XH_B8B-XH-A_1x08_P2.50mm_Vertical
- J3, J7, J8, J9, PWR-EXT-IN1: footprint Connector_JST:JST_XH_B2B-XH-AM_1x02_P2.50mm_Vertical -> Connector_JST:JST_XH_B2B-XH-A_1x02_P2.50mm_Vertical
- PWR-OUT3: footprint Connector_JST:JST_XH_B3B-XH-AM_1x03_P2.50mm_Vertical -> Connector_PinHeader_2.54mm:PinHeader_1x03_P2.54mm_Vertical
- VANILED1: footprint Connector_JST:JST_XH_B8B-XH-AM_1x08_P2.50mm_Vertical -> Connector_JST:JST_XH_B8B-XH-A_1x08_P2.50mm_Vertical
- moved T7 268.1 mm to (253.5, 99.2)
- moved COL1 255.3 mm to (222.8, 129.8), turned to 180 degrees
- moved COL2 249.4 mm to (228.8, 128.7)
- moved REG-COL2 240.0 mm to (238.5, 120.1)
- moved REG-COL1 238.2 mm to (217.8, 119.9)
- moved JP1 230.3 mm to (243.6, 67.9)
- moved J7 224.6 mm to (253.5, 94.2), turned to 90 degrees
- moved VANILED1 224.4 mm to (226.3, 54.4)
- moved J8 214.0 mm to (253.5, 85.6), turned to 90 degrees
- moved T2 204.9 mm to (207.3, 118.8)
- moved T1 204.6 mm to (191.4, 119.0)
- moved J9 204.0 mm to (253.5, 77.1), turned to 90 degrees
- moved CYBOARD-MACRO1 201.5 mm to (198.1, 123.4)
- moved J11 201.4 mm to (216.1, 88.4), turned to 180 degrees
- moved REG-ROW1 201.2 mm to (167.9, 117.1)
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Connections:
- C10 pad 1: +3V3 -> unconnected-(C10-Pad1)
- C10 pad 2: GND -> unconnected-(C10-Pad2)
- C19 pad 1: VCC -> +5V
- LED-LVL1 pad 6: VCC -> +5V
- R20 pad 1: +5V -> +3V3
- U1 pad 2: Serial-TX -> AUDIO
- U1 pad 3: Serial-RX -> /VBUS_DET
- U1 pad 38: AUDIO -> Net-(T5-Pin_1)
- U1 pad 39: Net-(T5-Pin_1) -> Net-(T6-Pin_1)
- U1 pad 40: /VBUS_DET -> Serial-TX
- U1 pad 41: Net-(T6-Pin_1) -> Serial-RX
- VANILED1 pad 3: VANILED_SIG1 -> VANILED_SIG4
- VANILED1 pad 4: VANILED_SIG2 -> VANILED_SIG3
- VANILED1 pad 5: VANILED_SIG3 -> VANILED_SIG2
- VANILED1 pad 6: VANILED_SIG4 -> VANILED_SIG1
Routing:
- net +5V: track 18.8 -> 102.6 mm, vias 2 -> 9
- net GND: track 72.8 -> 150.6 mm, vias 32 -> 50
- net VANILED_SIG1: track 4.59 -> 62.3 mm, vias 0 -> 1
- net VANILED_SIG4: track 4.08 -> 60.5 mm, vias 0 -> 1
- net VANILED_SIG2: track 4.42 -> 60.8 mm, vias 0 -> 1
- net VANILED_SIG3: track 4.25 -> 60.2 mm, vias 0 -> 1
- net AUDIO: track 3.91 -> 28.8 mm, vias 0 -> 3
- net /Serial_VBUS: track 0.00 -> 21.9 mm, vias 0 -> 2
- net Net-(J11-Pin_2): track 8.99 -> 27.0 mm
- net +3V3: track 109.2 -> 127.2 mm, vias 10 -> 12
- net Net-(J11-Pin_3): track 8.57 -> 25.3 mm
- net Serial-RX: track 14.6 -> 4.56 mm
- net LED_SCREEN_DI: track 0.00 -> 8.23 mm, vias 0 -> 2
- net Serial-TX: track 13.5 -> 5.54 mm
- net LED_SCREEN_DO: track 0.00 -> 7.66 mm, vias 0 -> 2
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
Commit message: even more progress, starting to come together.
Parts:
- J10, J5: footprint drawings:PinHeader_1x02_P1.27mm_Vertical -> Connector_PinSocket_2.54mm:PinSocket_1x02_P2.54mm_Vertical
- moved T3 80.1 mm to (169.9, 60.9)
- moved J10 75.3 mm to (200.1, 83.0), turned to 90 degrees
- moved J5 50.5 mm to (169.4, 75.3), turned to -90 degrees
- moved T9 20.8 mm to (106.8, 87.2)
- moved U11 20.3 mm to (191.6, 115.4), turned to 90 degrees
- moved U10 19.9 mm to (196.6, 115.4), turned to 90 degrees
- moved U12 19.0 mm to (199.1, 115.5), turned to 90 degrees
- moved U9 19.0 mm to (204.1, 115.5), turned to 90 degrees
- moved U13 18.8 mm to (194.1, 115.4), turned to 90 degrees
- moved R13 12.3 mm to (183.0, 97.5), turned to 90 degrees
- moved T1 9.37 mm to (182.6, 115.9)
- moved ROW1 9.09 mm to (174.6, 122.8)
- moved REG-ROW1 9.09 mm to (161.9, 110.2)
- moved C23 9.09 mm to (156.2, 107.2)
- moved PWR-OUT1 9.08 mm to (156.0, 69.2), turned to 90 degrees
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Connections:
- U1 pad 11: fal2-r2 -> rkjxt-a
- U1 pad 5: rkjxt-a -> fal2-r1
- U1 pad 6: rkjxt-b -> fal2-r2
- U1 pad 9: fal2-r1 -> rkjxt-b
Routing:
- net +5V: track 102.6 -> 213.8 mm, vias 9 -> 17
- net GND: track 150.6 -> 247.1 mm, vias 50 -> 79
- net fal1-r2: track 15.4 -> 87.4 mm, vias 0 -> 1
- net fal1-r1: track 15.2 -> 86.3 mm, vias 0 -> 1
- net LED_SCREEN_DI: track 8.23 -> 62.9 mm, vias 2 -> 3
- net LED_5V: track 0.00 -> 53.6 mm, vias 0 -> 2
- net fal2-r1: track 15.2 -> 66.5 mm, vias 0 -> 1
- net fal2-r2: track 19.6 -> 67.5 mm, vias 2 -> 1
- net LED_KEYS_DI: track 0.00 -> 40.2 mm, vias 0 -> 1
- net AUDIO: track 28.8 -> 55.3 mm
- net +3V3: track 127.2 -> 149.5 mm, vias 12 -> 13
- net LED_KEYBAR_DI: track 0.00 -> 19.7 mm
- net rkjxt-b: track 15.1 -> 34.4 mm, vias 0 -> 1
- net rkjxt-a: track 15.0 -> 31.6 mm, vias 0 -> 1
- net Net-(J4-Pin_4): track 0.00 -> 10.8 mm
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