File: mk19-rp2040.kicad_pcb (KiCad board)
At the start: 2 copper layers, 130 x 85 mm, 134 parts, among them J1 USB_C_Receptacle_USB2.0, J10 Conn_01x02, J11 Conn_01x03_Socket, J12 USB_C_Receptacle_USB2.0, J13 USB_C_Receptacle_USB2.0, J2 Conn_01x03_Socket, J3 Conn_01x02_Socket, J4 Conn_01x06_Socket, J5 Conn_01x02, J7 Conn_01x02_Socket, J8 Conn_01x02_Socket, J9 Conn_01x02_Socket, T1 Conn_01x01_Socket, T10 Conn_01x01_Socket, T11 Conn_01x01_Socket, T12 Conn_01x01_Socket, T13 Conn_01x01_Socket, T14 Conn_01x01_Socket, T15 Conn_01x01_Socket, T2 Conn_01x01_Socket, T3 Conn_01x01_Socket, T5 Conn_01x01_Socket, T6 Conn_01x01_Socket, T7 Conn_01x01_Socket, T9 Conn_01x01_Socket, U1 RP2040, U10 1N4148W_C81598, U11 1N4148W_C81598, U12 1N4148W_C81598, U13 1N4148W_C81598, U14 1N4148W_C81598, U15 1N4148W_C81598, U2 USBLC6-2P6, U3 XC6210B332MR-G, U4 USBLC6-2P6, U5 W25Q128JVS, U6 8_01A0_008200, U7 8_01A0_008200, U8 USBLC6-2P6, U9 1N4148W_C81598, Y1 Crystal_GND24

Commit message: almost done
Parts:
- LOGO1, LOGO2, LOGO3: moved to B.Cu
- moved LOGO7 150.5 mm to (175.0, 127.8)
- moved LOGO6 142.8 mm to (208.2, 127.8)
- moved T11 134.7 mm to (241.4, 84.9)
- moved LOGO3 130.2 mm to (250.3, 115.9), turned to 180 degrees
- moved LOGO1 129.1 mm to (141.8, 55.8), turned to 180 degrees
- moved T12 122.7 mm to (229.6, 92.0)
- moved LOGO4 122.7 mm to (142.0, 55.6)
- moved T13 119.7 mm to (228.7, 72.8)
- moved T14 117.3 mm to (225.2, 72.9)
- moved T9 112.7 mm to (218.6, 72.8)
- moved LOGO5 111.1 mm to (150.7, 51.4)
- moved T10 110.8 mm to (215.4, 72.7)
- moved T15 106.0 mm to (212.1, 72.8)
- moved LOGO2 92.4 mm to (150.4, 51.6), turned to 180 degrees
- moved COL_CS_MOS1 31.2 mm to (204.2, 95.5), turned to 180 degrees
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Connections:
- J12 pad A6: Split_Comms_RX -> Serial-RX
- J12 pad A7: Split_Comms_TX -> Serial-TX
- J12 pad B6: Split_Comms_RX -> Serial-RX
- J12 pad B7: Split_Comms_TX -> Serial-TX
- U8 pad 1: Split_Comms_RX -> Serial-RX
- U8 pad 3: Split_Comms_TX -> Serial-TX
- U8 pad 4: Split_Comms_TX -> Serial-TX
- U8 pad 6: Split_Comms_RX -> Serial-RX
Routing:
- net +3V3: track 149.5 -> 338.8 mm, vias 13 -> 35
- net col8: track 0.00 -> 186.2 mm, vias 0 -> 14
- net col7: track 0.00 -> 152.8 mm, vias 0 -> 16
- net SPI1_MOSI: track 6.90 -> 154.4 mm, vias 0 -> 8
- net +5V: track 213.8 -> 335.0 mm, vias 17 -> 29
- net SPI1_CLK: track 6.90 -> 123.3 mm, vias 0 -> 10
- net row4: track 0.00 -> 114.2 mm, vias 0 -> 7
- net GND: track 247.1 -> 354.8 mm, vias 79 -> 104
- net col6: track 0.00 -> 96.1 mm, vias 0 -> 10
- net LED_FAL1_DI: track 0.00 -> 90.4 mm, vias 0 -> 1
- net row2: track 0.00 -> 84.4 mm, vias 0 -> 7
- net row3: track 0.00 -> 84.0 mm, vias 0 -> 8
- net row5: track 0.00 -> 81.8 mm, vias 0 -> 8
- net col9: track 0.00 -> 71.4 mm, vias 0 -> 8
- net row0: track 0.00 -> 65.6 mm, vias 0 -> 2
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- added copper zone on F.Cu, net +5V
